Commit message: feat: create model parameter variables

File: urdf/articulated_bot.xacro (robot description, xacro)
@@ -2,4 +2,18 @@
 <robot name="udacity_bot" xmlns:xacro="http://www.ros.org/wiki/xacro">
   <xacro:include filename="$(find udacity_bot)/urdf/udacity_bot.gazebo" />
+  <xacro:property name="wheel_length" value="0.05" />
+  <xacro:property name="wheel_radius" value="0.1" />
+  <xacro:property name="wheel_mass" value="5" />
+  <xacro:property name="wheel_inertia" value="0.1" />
+  <xacro:property name="chassis_width" value="0.2" />
+  <xacro:property name="chassis_length" value="0.3" />
+  <xacro:property name="chassis_depth" value="0.1" />
+  <xacro:property name="chassis_mass" value="15" />
+  <xacro:property name="chassis_inertia" value="0.1" />
+  <xacro:property name="chassis_x_offset" value="${chassis_length/2 + 0.05}" />
+  <xacro:property name="wheel_x_offset" value="${chassis_x_offset + chassis_length/2 - wheel_radius}" />
+  <xacro:property name="wheel_y_offset" value="${(chassis_width + 0.1) / 2}" />
+  <xacro:property name="steer_angle_limit" value="0.95" />
+  <xacro:property name="steer_velocity" value="1" />
   <link name="robot_footprint"></link>
   <joint name="robot_footprint_joint" type="fixed">
@@ -10,27 +24,26 @@
   <!-- back chassis -->
   <link name='back_chassis'>
-    <pose>0 0 0.1 0 0 0</pose>
-    <inertial>
-      <mass value="15.0"/>
-      <origin xyz="0.0 0 0" rpy=" 0 0 0"/>
-      <inertia
-          ixx="0.1" ixy="0" ixz="0"
-          iyy="0.1" iyz="0"
-          izz="0.1" />
+    <inertial>
+      <mass value="${chassis_mass}"/>
+      <origin xyz="-${chassis_x_offset} 0 0" rpy=" 0 0 0"/>
+      <inertia
+          ixx="${chassis_inertia}" ixy="0" ixz="0"
+          iyy="${chassis_inertia}" iyz="0"
+          izz="${chassis_inertia}" />
     </inertial>
     <collision name='collision'>
-      <origin xyz="0 0 0" rpy=" 0 0 0"/>
-      <geometry>
-        <box size=".4 .2 .1"/>
+      <origin xyz="-${chassis_x_offset} 0 0" rpy=" 0 0 0"/>
+      <geometry>
+        <box size="${chassis_length} ${chassis_width} ${chassis_depth}"/>
       </geometry>
     </collision>
     <visual name='chassis_visual'>
-      <origin xyz="0 0 0" rpy=" 0 0 0"/>
-      <geometry>
-        <box size=".4 .2 .1"/>
+      <origin xyz="-${chassis_x_offset} 0 0" rpy=" 0 0 0"/>
+      <geometry>
+        <box size="${chassis_length} ${chassis_width} ${chassis_depth}"/>
       </geometry>
     </visual>
     <visual name='back_chassis_link_visual'>
-      <origin xyz="0.225 0 0" rpy=" 0 0 0"/>
+      <origin xyz="-0.025 0 0" rpy=" 0 0 0"/>
       <geometry>
         <box size=".05 .01 .05"/>
@@ -38,5 +51,5 @@
     </visual>
     <visual name='chassis_pin_visual'>
-      <origin xyz="0.25 0 0" rpy=" 0 0 0"/>
+      <origin xyz="0 0 0" rpy=" 0 0 0"/>
       <geometry>
         <cylinder length="0.06" radius="0.025"/>
@@ -46,15 +59,15 @@
   <link name="left_wheel">
     <inertial>
-      <mass value="5.0"/>
-      <origin xyz="0.0 0 0" rpy=" 0 1.5707 1.5707"/>
-      <inertia
-          ixx="0.1" ixy="0" ixz="0"
-          iyy="0.1" iyz="0"
-          izz="0.1" />
+      <mass value="${wheel_mass}"/>
+      <origin xyz="0 0 0" rpy=" 0 1.5707 1.5707"/>
+      <inertia
+          ixx="${wheel_inertia}" ixy="0" ixz="0"
+          iyy="${wheel_inertia}" iyz="0"
+          izz="${wheel_inertia}" />
     </inertial>
     <collision name="left_wheel_collision">
       <origin xyz="0 0 0" rpy=" 0 1.5707 1.5707"/>
       <geometry>
-        <cylinder length="0.05" radius="0.1"/>
+        <cylinder length="${wheel_length}" radius="${wheel_radius}"/>
       </geometry>
     </collision>
@@ -62,10 +75,10 @@
       <origin xyz="0 0 0" rpy=" 0 1.5707 1.5707"/>
       <geometry>
-        <cylinder length="0.05" radius="0.1"/>
+        <cylinder length="${wheel_length}" radius="${wheel_radius}"/>
       </geometry>
     </visual>
   </link>
   <joint type="continuous" name="left_wheel_hinge">
-    <origin xyz="-0.1 0.15 0" rpy="0 0 0"/>
+    <origin xyz="-${wheel_x_offset}  ${wheel_y_offset} 0" rpy="0 0 0"/>
     <child link="left_wheel"/>
     <parent link="back_chassis"/>
@@ -76,15 +89,15 @@
   <link name="right_wheel">
     <inertial>
-      <mass value="5.0"/>
+      <mass value="${wheel_mass}"/>
       <origin xyz="0.0 0 0" rpy=" 0 1.5707 1.5707"/>
       <inertia
-          ixx="0.1" ixy="0" ixz="0"
-          iyy="0.1" iyz="0"
-          izz="0.1" />
+          ixx="${wheel_inertia}" ixy="0" ixz="0"
+          iyy="${wheel_inertia}" iyz="0"
+          izz="${wheel_inertia}" />
     </inertial>
     <collision name="right_wheel_collision">
       <origin xyz="0 0 0" rpy=" 0 1.5707 1.5707"/>
       <geometry>
-        <cylinder length="0.05" radius="0.1"/>
+        <cylinder length="${wheel_length}" radius="${wheel_radius}"/>
       </geometry>
     </collision>
@@ -92,10 +105,10 @@
       <origin xyz="0 0 0" rpy=" 0 1.5707 1.5707"/>
       <geometry>
-        <cylinder length="0.05" radius="0.1"/>
+        <cylinder length="${wheel_length}" radius="${wheel_radius}"/>
       </geometry>
     </visual>
   </link>
   <joint type="continuous" name="right_wheel_hinge">
-    <origin xyz="-0.1 -0.15 0" rpy="0 0 0"/>
+    <origin xyz="-${wheel_x_offset} -${wheel_y_offset} 0" rpy="0 0 0"/>
     <child link="right_wheel"/>
     <parent link="back_chassis"/>
@@ -106,31 +119,30 @@
   <!-- front chassis -->
   <joint type="revolute" name="chassis_hinge">
-    <origin xyz="0.25 0 0" rpy="0 0 0"/>
+    <origin xyz="0 0 0" rpy="0 0 0"/>
     <child link="front_chassis"/>
     <parent link="back_chassis"/>
     <axis xyz="0 0 1" rpy="0 0 0"/>
-    <limit effort="10000" lower="-1" upper="1" velocity="1"/>
+    <limit effort="10000" lower="-${steer_angle_limit}" upper="${steer_angle_limit}" velocity="${steer_velocity}"/>
     <joint_properties damping="1.0" friction="1.0"/>
   </joint>
   <link name='front_chassis'>
-    <pose>0.05 0 0.1 0 0 0</pose>
-    <inertial>
-      <mass value="15.0"/>
-      <origin xyz="0.25 0 0" rpy=" 0 0 0"/>
-      <inertia
-          ixx="0.1" ixy="0" ixz="0"
-          iyy="0.1" iyz="0"
-          izz="0.1" />
+    <inertial>
+      <mass value="${chassis_mass}"/>
+      <origin xyz="${chassis_x_offset} 0 0" rpy=" 0 0 0"/>
+      <inertia
+          ixx="${chassis_inertia}" ixy="0" ixz="0"
+          iyy="${chassis_inertia}" iyz="0"
+          izz="${chassis_inertia}" />
     </inertial>
     <collision name='collision'>
-      <origin xyz="0.25 0 0" rpy=" 0 0 0"/>
-      <geometry>
-        <box size=".4 .2 .1"/>
+      <origin xyz="${chassis_x_offset} 0 0" rpy=" 0 0 0"/>
+      <geometry>
+        <box size="${chassis_length} ${chassis_width} ${chassis_depth}"/>
       </geometry>
     </collision>
     <visual name='chassis_visual'>
-      <origin xyz="0.25 0 0" rpy=" 0 0 0"/>
-      <geometry>
-        <box size=".4 .2 .1"/>
+      <origin xyz="${chassis_x_offset} 0 0" rpy=" 0 0 0"/>
+      <geometry>
+        <box size="${chassis_length} ${chassis_width} ${chassis_depth}"/>
       </geometry>
     </visual>
@@ -144,15 +156,15 @@
   <link name="left_front_wheel">
     <inertial>
-      <mass value="5.0"/>
+      <mass value="${wheel_mass}"/>
       <origin xyz="0.0 0 0" rpy=" 0 1.5707 1.5707"/>
       <inertia
-          ixx="0.1" ixy="0" ixz="0"
-          iyy="0.1" iyz="0"
-          izz="0.1" />
+          ixx="${wheel_inertia}" ixy="0" ixz="0"
+          iyy="${wheel_inertia}" iyz="0"
+          izz="${wheel_inertia}" />
     </inertial>
     <collision name="collision">
       <origin xyz="0 0 0" rpy=" 0 1.5707 1.5707"/>
       <geometry>
-        <cylinder length="0.05" radius="0.1"/>
+        <cylinder length="${wheel_length}" radius="${wheel_radius}"/>
       </geometry>
     </collision>
@@ -160,10 +172,10 @@
       <origin xyz="0 0 0" rpy=" 0 1.5707 1.5707"/>
       <geometry>
-        <cylinder length="0.05" radius="0.1"/>
+        <cylinder length="${wheel_length}" radius="${wheel_radius}"/>
       </geometry>
     </visual>
   </link>
   <joint type="continuous" name="left_front_wheel_hinge">
-    <origin xyz="0.35 0.15 0" rpy="0 0 0"/>
+    <origin xyz="${wheel_x_offset} ${wheel_y_offset} 0" rpy="0 0 0"/>
     <child link="left_front_wheel"/>
     <parent link="front_chassis"/>
@@ -174,15 +186,15 @@
   <link name="right_front_wheel">
     <inertial>
-      <mass value="5.0"/>
+      <mass value="${wheel_mass}"/>
       <origin xyz="0.0 0 0" rpy=" 0 1.5707 1.5707"/>
       <inertia
-          ixx="0.1" ixy="0" ixz="0"
-          iyy="0.1" iyz="0"
-          izz="0.1" />
+          ixx="${wheel_inertia}" ixy="0" ixz="0"
+          iyy="${wheel_inertia}" iyz="0"
+          izz="${wheel_inertia}" />
     </inertial>
     <collision name="collision">
       <origin xyz="0 0 0" rpy=" 0 1.5707 1.5707"/>
       <geometry>
-        <cylinder length="0.05" radius="0.1"/>
+        <cylinder length="${wheel_length}" radius="${wheel_radius}"/>
       </geometry>
     </collision>
@@ -190,10 +202,10 @@
       <origin xyz="0 0 0" rpy=" 0 1.5707 1.5707"/>
       <geometry>
-        <cylinder length="0.05" radius="0.1"/>
+        <cylinder length="${wheel_length}" radius="${wheel_radius}"/>
       </geometry>
     </visual>
   </link>
   <joint type="continuous" name="right_front_wheel_hinge">
-    <origin xyz="0.35 -0.15 0" rpy="0 0 0"/>
+    <origin xyz="${wheel_x_offset} -${wheel_y_offset} 0" rpy="0 0 0"/>
     <child link="right_front_wheel"/>
     <parent link="front_chassis"/>
@@ -226,5 +238,5 @@
   </link>
   <joint type="fixed" name="camera_joint">
-    <origin xyz="0.45 0 0" rpy="0 0 0"/>
+    <origin xyz="${chassis_x_offset + chassis_length/2} 0 0" rpy="0 0 0"/>
     <child link="camera"/>
     <parent link="front_chassis"/>
@@ -235,5 +247,4 @@
   <!-- laser -->
   <link name='hokuyo'>
-    <pose>0 0 0 0 0 0</pose>
     <inertial>
       <mass value="0.1"/>
@@ -258,5 +269,5 @@
   </link>
   <joint type="fixed" name="hokuyo_joint">
-    <origin xyz="0.15 0 0.1" rpy="0 0 0"/>
+    <origin xyz="${chassis_x_offset} 0 ${wheel_radius + 0.01}" rpy="0 0 0"/>
     <child link="hokuyo"/>
     <parent link="front_chassis"/>
